File: doc/ESP-NOW-RC-Car/ESP-NOW-RC-Car.kicad_sch (KiCad schematic)
At the start: 10 parts, among them M1 Motor_DC, M2 Motor_DC, M3 Motor_DC, M4 Motor_DC, P1 USB_C_Plug_USB2.0, U1 ESP32-WROOM-32, U2 L298N, U3 L298N

Commit message: update(CAD): files
WIP

#4
Connections:
- net at P1.A1 (GND), P1.A12 (GND), P1.B1 (GND)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: now also BT1.2 (-), BT2.2 (-), U1.1 (GND), U1.15 (GND), U1.38 (GND), U1.39 (GND), U2.8 (GND), U3.8 (GND)
- net at P1.A4 (VBUS), P1.A9 (VBUS), P1.B4 (VBUS)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: now also U1.2 (VDD), U2.9 (Vss)
- net at U3.4 (Vs): now also BT1.1 (+)
- net at U2.4 (Vs): now also BT2.1 (+)
